File: hardware/ima/interface.kicad_sch (KiCad schematic)
At the start: 10 parts, among them J3 USB_B_Mini, SW2 RotaryEncoder_Switch, U7 SD Card SDIO Breakout, U8 NUCLEO STM32F401re, U9 SH1107_128x128

Commit message: add schematics to .tex
Parts:
- removed J3: USB_B_Mini, symbol Connector:USB_B_Mini
- removed RV10: Fader 1, symbol Device:R_Potentiometer
- removed RV6: Fader 5, symbol Device:R_Potentiometer
- removed RV7: Fader 4, symbol Device:R_Potentiometer
- removed RV8: Fader 3, symbol Device:R_Potentiometer
- removed RV9: Fader 2, symbol Device:R_Potentiometer
- removed SW2: RotaryEncoder_Switch, symbol Device:RotaryEncoder_Switch
- removed U7: SD Card SDIO Breakout, symbol New_Library:Waveshare_SD_Card_Breakout
- removed U8: NUCLEO STM32F401re, Package_QFP:LQFP-64_10x10mm_P0.5mm, symbol MCU_ST_STM32F4:STM32F401RETx
- removed U9: SH1107_128x128, symbol New_Library:128x128Display
- added J4: USB_B_Mini, symbol Connector:USB_B_Mini
- added RV1: Fader 1, symbol Device:R_Potentiometer
- added RV2: Fader 2, symbol Device:R_Potentiometer
- added RV3: Fader 3, symbol Device:R_Potentiometer
- added RV4: Fader 4, symbol Device:R_Potentiometer
- added RV5: Fader 5, symbol Device:R_Potentiometer
- added SW1: RotaryEncoder_Switch, symbol Device:RotaryEncoder_Switch
- added U4: SD Card SDIO Breakout, symbol New_Library:Waveshare_SD_Card_Breakout
- added U5: SH1107_128x128, symbol New_Library:128x128Display
- added U6: NUCLEO STM32F401re, Package_QFP:LQFP-64_10x10mm_P0.5mm, symbol MCU_ST_STM32F4:STM32F401RETx
Connections:
- net +3V3: now also RV1.1, RV2.1, RV3.1, RV4.1, RV5.1, U4.9 (3.3V), U5.4 (VCC), U6.65 (3v3)
- net +5V: now also J4.1 (VBUS), U6.18 (VSS), U6.31 (VSS), U6.47 (VSS), U6.63 (VSS)
- net GND: now also RV1.3, RV2.3, RV3.3, RV4.3, RV5.3, SW1.C, SW1.S2, U4.8 (GND), U5.3 (GND)
- new net: RV5.2, U6.8 (PC0)
- new net: RV3.2, U6.23 (PA7)
- new net: U4.2 (D1), U6.40 (PC9)
- new net: U4.3 (D2), U6.51 (PC10)
- new net: U4.4 (D3), U6.52 (PC11)
- new net: U4.5 (CLK), U6.53 (PC12)
- new net: U4.6 (CMD), U6.54 (PD2)
- new net: U4.7 (D0), U6.39 (PC8)
- new net: RV1.2, U6.21 (PA5)
- new net: RV4.2, U6.41 (PA8)
- new net: SW1.A, U6.14 (PA0)
- new net: SW1.B, U6.15 (PA1)
- new net: J4.5 (GND), J4.6 (Shield), U6.19 (VDD), U6.32 (VDD), U6.48 (VDD), U6.64 (VDD)
- new net: SW1.S1, U6.20 (PA4)
- new net: RV2.2, U6.22 (PA6)
- new net: U5.2 (SCL), U6.58 (PB6)
- new net: U5.1 (SDA), U6.59 (PB7)
